File: elec/layout/default/saleae-header.kicad_pcb (KiCad board)
At the start: 2 copper layers, 225.7 x 100.8 mm, 0 parts

Commit message: layout
Parts:
- added R1: Chip Resistor - Surface Mount 1KOhms ±5% 1/16W 0402 RoHS, lib:R0402, F.Cu at (130.0, 59.9)
- added R2: Chip Resistor - Surface Mount 1KOhms ±5% 1/16W 0402 RoHS, lib:R0402, F.Cu at (132.5, 59.9)
- added R3: Chip Resistor - Surface Mount 1KOhms ±5% 1/16W 0402 RoHS, lib:R0402, F.Cu at (135.1, 59.9)
- added R4: Chip Resistor - Surface Mount 1KOhms ±5% 1/16W 0402 RoHS, lib:R0402, F.Cu at (137.6, 59.9)
- added U1: , lib:HDR-SMD_8P-P2.54-V-M-R2-C4-LS7.4, F.Cu at (133.8, 54.3)
Routing:
- net gnd: track 0.00 -> 7.62 mm
- net _1: track 0.00 -> 2.29 mm
- net _3: track 0.00 -> 2.29 mm
- net _5: track 0.00 -> 2.29 mm
- net _7: track 0.00 -> 2.28 mm
